File: kicad/C64 RS232 Adapter Board - v1/C64 RS232 Adapter Board.sch (KiCad schematic (older format))
At the start: 29 parts, among them J1 RS232_HDR, J2 DB25_RS232, J3 C64_USER_PORT, J4 User Port Breakout, SW1 RESET, U1 MAX3241ECAI+T

Commit message: added vias
Parts:
- removed D2: 232-PWR, LED_SMD:LED_1206_3216Metric_Pad1.42x1.75mm_HandSolder, symbol Device:LED_Small
- removed H5, H6, H? (x2): MountingHole, MountingHole:MountingHole_2.5mm, symbol Mechanical:MountingHole
- removed R3: 1K, Resistor_SMD:R_0805_2012Metric_Pad1.15x1.40mm_HandSolder, symbol Device:R_Small
- added JP10, JP11, JP2, JP3, JP4, JP5, JP7, JP9: SolderJumper_2_Bridged, Jumper:SolderJumper-2_P1.3mm_Bridged_RoundedPad1.0x1.5mm, symbol Jumper:SolderJumper_2_Bridged
- C1, C2, C3, C4, C5: footprint Capacitor_SMD:C_0805_2012Metric_Pad1.15x1.40mm_HandSolder -> Capacitor_SMD:C_0805_2012Metric
- D1: value C64-PWR -> PWR; footprint LED_SMD:LED_1206_3216Metric_Pad1.42x1.75mm_HandSolder -> LED_SMD:LED_1206_3216Metric
- J4: footprint My Libraries:C64_2.54mm_User_Port -> My Libraries:TSM-for-C64-User-Port; MFN (none) -> 15-91-0240; Manu (none) -> Molex; SPN (none) -> 25M0665
- JP1, JP6, JP8: footprint Jumper:SolderJumper-2_P1.3mm_Open_TrianglePad1.0x1.5mm -> Jumper:SolderJumper-2_P1.3mm_Bridged_RoundedPad1.0x1.5mm; symbol Jumper:SolderJumper_2_Open -> Jumper:SolderJumper_2_Bridged
- R1, R2: footprint Resistor_SMD:R_0805_2012Metric_Pad1.15x1.40mm_HandSolder -> Resistor_SMD:R_0805_2012Metric
Connections:
- wire segments 108 -> 116
Other:
- moved on the sheet: J1
